File: rhythmpad/rhythmpad.kicad_sch (KiCad schematic)
At the start: 20 parts, among them SW1 SW_Push, SW10 SW_Push, SW2 SW_Push, SW3 SW_Push, SW4 SW_Push, SW5 SW_Push, SW6 SW_Push, SW7 SW_Push, SW8 SW_Push, SW9 SW_Push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

Commit message: commit pcb/schematic changes
Parts:
- added D11, D12, D13, D14: SK6812MINI, LED_SMD:LED_SK6812MINI_PLCC4_3.5x3.5mm_P1.75mm, symbol LED:SK6812MINI
- added D7: D, Diode_THT:D_DO-35_SOD27_P7.62mm_Horizontal, symbol Device:D
- D1: renamed from D2; footprint (none) -> Diode_THT:D_DO-35_SOD27_P7.62mm_Horizontal
- D10, D8, D9: footprint (none) -> Diode_THT:D_DO-35_SOD27_P7.62mm_Horizontal
- D2: renamed from D3; footprint (none) -> Diode_THT:D_DO-35_SOD27_P7.62mm_Horizontal
- D3: renamed from D4; footprint (none) -> Diode_THT:D_DO-35_SOD27_P7.62mm_Horizontal
- D4: renamed from D5; footprint (none) -> Diode_THT:D_DO-35_SOD27_P7.62mm_Horizontal
- D5: renamed from D6; footprint (none) -> Diode_THT:D_DO-35_SOD27_P7.62mm_Horizontal
- D6: renamed from D7; footprint (none) -> Diode_THT:D_DO-35_SOD27_P7.62mm_Horizontal
- SW1, SW10, SW2, SW3, SW4, SW5, SW6, SW7, SW8, SW9: footprint (none) -> Button_Switch_Keyboard:SW_Cherry_MX_1.00u_PCB
- U1: footprint Module:MOUDLE14P-XIAO-DIP-SMD -> OPL:XIAO-RP2040-DIP
Connections:
- net Col 0: now also U1.4 (GPIO29/ADC3/A3); no longer U1.11 (GPIO3/MOSI)
- net Col 1: now also U1.5 (GPIO6/SDA); no longer U1.10 (GPIO4/MISO)
- net Col 2: now also U1.6 (GPIO7/SCL); no longer U1.5 (GPIO6/SDA)
- net GND: now also D11.2 (VSS), D12.2 (VSS), D13.2 (VSS), D14.2 (VSS); no longer SW7.1
- net Row 0: now also U1.8 (GPIO1/RX); no longer U1.7 (GPIO0/TX)
- net Row 1: now also U1.9 (GPIO2/SCK), D7.1 (K); no longer U1.8 (GPIO1/RX)
- net Row 2: now also U1.10 (GPIO4/MISO); no longer U1.9 (GPIO2/SCK)
- net Col 3: now reaches SW7.2
- net Col 3: now also U1.7 (GPIO0/TX); no longer U1.6 (GPIO7/SCL)
- net at U1.1 (GPIO26/ADC0/A0): now also D12.1 (DOUT)
- net +5V: now reaches U1.14 (VBUS)
- net +5V: now also D11.4 (VDD), D12.4 (VDD), D13.4 (VDD), D14.4 (VDD)
- new net: D7.2 (A), SW7.1
- new net: D14.1 (DOUT), U1.11 (GPIO3/MOSI)
- new net: D13.1 (DOUT), D14.3 (DIN)
- new net: D11.1 (DOUT), D12.3 (DIN)
Other:
- moved on the sheet: SW7
