File: rhythmpad/rhythmpad.kicad_pcb (KiCad board)
At the start: 2 copper layers, 90.5 x 76.2 mm, 25 parts, among them SW1 SW_Push, SW10 SW_Push, SW2 SW_Push, SW3 SW_Push, SW4 SW_Push, SW5 SW_Push, SW6 SW_Push, SW7 SW_Push, SW8 SW_Push, SW9 SW_Push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

Commit message: add library/finish pcb
Other:
- board text added: "XIAO HERE!"
- board text added: "mikael's rhythmpad"
